Commit message: Add files via upload

File: src/my_azu/my_azu/urdf/azu.urdf.xacro (robot description, xacro)
@@ -65,13 +65,5 @@
       <inertia ixx="0.001" ixy="0" ixz="0" iyy="0.001" iyz="0" izz="0.001" />
     </inertial>
-    <visual>
-      <origin xyz="0.0 0.0 0.0" rpy="0 0 0" />
-      <geometry>
-        <box size="0.08 0.08 0.08" />
-      </geometry>
-      <material name="gray">
-        <color rgba="0.5 0.5 0.5 1.0" />
-      </material>
-    </visual>
+    <!-- Visual: không hiển thị (đã nằm trong Head mesh) -->
     <collision>
       <origin xyz="0.0 0.0 0.0" rpy="0 0 0" />
@@ -88,13 +80,5 @@
       <inertia ixx="0.01" ixy="0" ixz="0" iyy="0.01" iyz="0" izz="0.01" />
     </inertial>
-    <visual>
-      <origin xyz="0.0 0.0 0.0" rpy="0 0 0" />
-      <geometry>
-        <cylinder radius="0.05" length="0.10" />
-      </geometry>
-      <material name="black">
-        <color rgba="0.0 0.0 0.0 1.0" />
-      </material>
-    </visual>
+    <!-- Visual: không hiển thị (đã nằm trong Head mesh) -->
     <collision>
       <origin xyz="0.0 0.0 0.0" rpy="0 0 0" />
